File: makyi_mouse.kicad_sch (KiCad schematic)
At the start: 70 parts, among them J1 Conn_01x02_Pin, J10 Conn_01x06_Pin, J12 Conn_01x06_Pin, J14 20021221-00006C4LF, J3 Conn_01x04_Pin, J5 Conn_01x04_Pin, J6 Conn_01x04_Pin, J8 Conn_01x04_Pin, M1 Motor_DC, M2 Motor_DC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

Commit message: 壁センサ修正
Parts:
- renumbered Q1 to Q2
